File: boards/relay8/relay8.kicad_pcb (KiCad board)
At the start: 2 copper layers, 232 x 110 mm, 60 parts, among them J1 USB-C, J11 CH1, J12 CH2, J13 CH3, J14 CH4, J15 CH5, J16 CH6, J17 CH7, J18 CH8, J2 UART, J20 MAINS IN, K1 SRD-05VDC-SL-C, K2 SRD-05VDC-SL-C, K3 SRD-05VDC-SL-C, K4 SRD-05VDC-SL-C, K5 SRD-05VDC-SL-C, K6 SRD-05VDC-SL-C, K7 SRD-05VDC-SL-C, K8 SRD-05VDC-SL-C, SW1 RESET, SW2 BOOT, U1 ESP32-C3-WROOM-02-N4, U2 LP38693MP-3.3, U3 ULN2803A

Commit message: relay8: VBUS soft-start (AO3401A) keeps USB hot-plug inrush within USB 2.0
Parts:
- added C6: 100nF, Capacitor_SMD:C_0402_1005Metric, F.Cu at (159.0, 193.5)
- added C7: 10nF, Capacitor_SMD:C_0402_1005Metric, F.Cu at (162.5, 191.5)
- added C8: 1uF, Capacitor_SMD:C_0402_1005Metric, F.Cu at (167.0, 195.5)
- added Q1: AO3401A, Package_TO_SOT_SMD:SOT-23, F.Cu at (155.0, 192.5)
- added R9: 100k, Resistor_SMD:R_0402_1005Metric, F.Cu at (159.0, 191.5)
Connections:
- D5 pad 2: VBUS -> VSW
Routing:
- net VSW: track 0.00 -> 20.5 mm, vias 0 -> 3
- net +3V3: track 175.5 -> 194.7 mm, vias 4 -> 3
- net EN: track 116.3 -> 129.3 mm, vias 0 -> 2
- net SS_G: track 0.00 -> 12.0 mm
- net RLY7: track 88.7 -> 76.9 mm, vias 1 -> 0
- net TXD: track 69.9 -> 59.9 mm
- net IO9: track 113.3 -> 104.7 mm
- net VBUS: track 56.0 -> 48.0 mm, vias 4 -> 2
- net GND: track 310.5 -> 318.5 mm, vias 5 -> 7
- net RLY5: track 32.8 -> 40.5 mm
- net 5V_PS: track 367.2 -> 374.6 mm
- net RLY8: track 100.0 -> 106.3 mm
- net IN5: track 86.5 -> 92.8 mm
- net RXD: track 67.2 -> 61.5 mm, vias 1 -> 0
- net IN2: track 73.4 -> 77.3 mm
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