File: boards/relay8/relay8.kicad_sch (KiCad schematic)
At the start: 65 parts, among them J1 USB-C, J11 CH1, J12 CH2, J13 CH3, J14 CH4, J15 CH5, J16 CH6, J17 CH7, J18 CH8, J2 UART, J20 MAINS IN, K1 SRD-05VDC-SL-C, K2 SRD-05VDC-SL-C, K3 SRD-05VDC-SL-C, K4 SRD-05VDC-SL-C, K5 SRD-05VDC-SL-C, K6 SRD-05VDC-SL-C, K7 SRD-05VDC-SL-C, K8 SRD-05VDC-SL-C, Q1 AO3401A, SW1 RESET, SW2 BOOT, U1 ESP32-C3-WROOM-02-N4, U2 LP38693MP-3.3, U3 ULN2803A

Commit message: cm5: two 802.3at PoE ports (IP804AR PSE, G2423S magnetics, RJHSE5380) on the LAN7800s
IP804AR in auto mode without EEPROM, ports 0/1, Alternative A. G2423S
footprint generated from the datasheet land pattern; IP804AR symbol
matches the datasheet pin table 48/48. rails.json declares the 54 V
input range so review.py can check V54 against 802.3at (50-57 V); two
new mutations are caught.

netlabel: no NC flag on pins whose electrical type is already
no_connect (KiCad reported one as dangling). relay8 loses one redundant
flag; its ERC and netlist are unchanged.
Connections:
- no-connect marks 3 -> 2
Changed lines of the file:
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@@
 		(at 46.99 91.44)
-	)
-	(no_connect
-		(at 134.62 38.1)
 	)
 	(global_label "VBUS"
