File: boards/cm5/cm5.kicad_sch (KiCad schematic)
At the start: 36 parts, among them J20 54V IN, Q10 BSC160N10NS3G, Q11 BSC070N10NS5, U10 LM5146RGYR

Commit message: cm5: 5 V -> 3.3 V / 8 A (TPS568230), enabled by the 5 V power-good through a divider
Values from the TPS568230 datasheet table 3 (3.3 V, 600 kHz, 1.5 uH) and
table 1 (MODE 330k/5.1k = Eco-mode). EN is rated 4 V max, so the LM5146
PGOOD pull-up to 5 V is divided to 3.0 V. ERC 0, netlist 152/152, review
0 errors.
Parts:
- added C40, C41, C42, C43, C45, C46: 47uF, Capacitor_SMD:C_1210_3225Metric, symbol Device:C
- added C44: 100pF, Capacitor_SMD:C_0402_1005Metric, symbol Device:C
- added C47, C49: 100nF, Capacitor_SMD:C_0402_1005Metric, symbol Device:C
- added C48: 1uF, Capacitor_SMD:C_0402_1005Metric, symbol Device:C
- added L20: 1.5uH IHLP4040, Inductor_SMD:L_Vishay_IHLP-4040, symbol Device:L
- added R19: 30k, Resistor_SMD:R_0402_1005Metric, symbol Device:R
- added R21: 91k, Resistor_SMD:R_0402_1005Metric, symbol Device:R
- added R22: 20k, Resistor_SMD:R_0402_1005Metric, symbol Device:R
- added R23: 330k, Resistor_SMD:R_0402_1005Metric, symbol Device:R
- added R24: 5.1k, Resistor_SMD:R_0402_1005Metric, symbol Device:R
- added R25: 100k, Resistor_SMD:R_0402_1005Metric, symbol Device:R
- added U20: TPS568230RJER, Package_DFN_QFN:Texas_RJE0020A_VQFN-20-1EP_3x3mm_P0.45mm_EP0.675x0.76mm, symbol Regulator_Switching:TPS568230
Connections:
- net +5V: now also C45.1, C46.1, C47.1, U20.2 (VIN), U20.3 (VIN), U20.4 (VIN), U20.5 (VIN)
- net GND: now also C40.2, C41.2, C42.2, C43.2, C45.2, C46.2, C47.2, C48.2, R19.2, R22.2, R24.2, U20.13 (AGND), U20.18 (GND), U20.21 (GND), U20.7 (GND), U20.8 (GND)
- net PG_5V: now also R19.1, U20.12 (EN)
- new net: U20.10 (NC), U20.16 (NC)
- new net +3V3: C40.1, C41.1, C42.1, C43.1, C44.1, L20.2, R21.1, R25.1
- new net BST3: C49.1, U20.1 (BST)
- new net FB3: C44.2, R21.2, R22.1, U20.14 (FB)
- new net MODE3: R23.2, R24.1, U20.15 (MODE)
- new net PG_3V3: R25.2, U20.9 (PGOOD)
- new net SW3: C49.2, L20.1, U20.19 (SW), U20.20 (SW), U20.6 (SW)
- new net VCC3: C48.1, R23.1, U20.17 (VCC)
- no-connect marks 3 -> 5

Commit message: cm5: CM5 connector power, GPIO_VREF, RTC battery, buttons and LEDs; +3V3 now follows CM5_3V3
+3V3 is enabled by the LM5146 power-good pulled up to CM5_3V3, so the
peripheral rail is on only while the module is on and cannot back-feed
it (CM5 datasheet 3.1). Remaining CM5 pins are no-connect until their
blocks are added. Sheet is A1.

review.py: LEDs with the resistor on the cathode side, supply pins tied
to GND, and supply pins with no decoupling requirement. Two new cm5
mutations; all mutation tests pass and the other boards' reviews are
unchanged.
Parts:
- removed U20: TPS568230RJER, Package_DFN_QFN:Texas_RJE0020A_VQFN-20-1EP_3x3mm_P0.45mm_EP0.675x0.76mm, symbol Regulator_Switching:TPS568230
- added BT50: CR2032, Battery:BatteryHolder_Keystone_3034_1x20mm, symbol Device:Battery_Cell
- added C45, C50: 47uF, Capacitor_SMD:C_1210_3225Metric, symbol Device:C
- added C51: 100nF, Capacitor_SMD:C_0402_1005Metric, symbol Device:C
- added D50: RED, LED_SMD:LED_0805_2012Metric, symbol Device:LED
- added D51: GREEN, LED_SMD:LED_0805_2012Metric, symbol Device:LED
- added J2: CM5 pins 101-200, CM5:Amphenol_10164227-1001A1RLF_2x50_P0.4mm, symbol CM5:CM5_J2
- added R50, R51: 1k, Resistor_SMD:R_0402_1005Metric, symbol Device:R
- added SW50: POWER, Button_Switch_SMD:SW_Push_1P1T_NO_CK_KMR2, symbol Switch:SW_Push
- added SW51: RPIBOOT, Button_Switch_SMD:SW_Push_1P1T_NO_CK_KMR2, symbol Switch:SW_Push
- C40: renamed from R22; value 20k -> 47uF; footprint Resistor_SMD:R_0402_1005Metric -> Capacitor_SMD:C_1210_3225Metric; symbol Device:R -> Device:C
- C44: renamed from R21; value 91k -> 100pF; footprint Resistor_SMD:R_0402_1005Metric -> Capacitor_SMD:C_0402_1005Metric; symbol Device:R -> Device:C
- C47: renamed from C46; value 47uF -> 100nF; footprint Capacitor_SMD:C_1210_3225Metric -> Capacitor_SMD:C_0402_1005Metric
- C48: renamed from C47; value 100nF -> 1uF
- C49: renamed from R24; value 5.1k -> 100nF; footprint Resistor_SMD:R_0402_1005Metric -> Capacitor_SMD:C_0402_1005Metric; symbol Device:R -> Device:C
- J1: renamed from R25; value 100k -> CM5 pins 1-100; footprint Resistor_SMD:R_0402_1005Metric -> CM5:Amphenol_10164227-1001A1RLF_2x50_P0.4mm; symbol Device:R -> CM5:CM5_J1
- L20: renamed from C49; value 100nF -> 1.5uH IHLP4040; footprint Capacitor_SMD:C_0402_1005Metric -> Inductor_SMD:L_Vishay_IHLP-4040; symbol Device:C -> Device:L
- R18: value 20k -> 10k
- R21: renamed from L20; value 1.5uH IHLP4040 -> 91k; footprint Inductor_SMD:L_Vishay_IHLP-4040 -> Resistor_SMD:R_0402_1005Metric; symbol Device:L -> Device:R
- R22: renamed from C44; value 100pF -> 20k; footprint Capacitor_SMD:C_0402_1005Metric -> Resistor_SMD:R_0402_1005Metric; symbol Device:C -> Device:R
- R23: renamed from C48; value 1uF -> 330k; footprint Capacitor_SMD:C_0402_1005Metric -> Resistor_SMD:R_0402_1005Metric; symbol Device:C -> Device:R
- R24: renamed from R23; value 330k -> 5.1k
- R25: renamed from C43; value 47uF -> 100k; footprint Capacitor_SMD:C_1210_3225Metric -> Resistor_SMD:R_0402_1005Metric; symbol Device:C -> Device:R
- U20: renamed from R19; value 30k -> TPS568230RJER; footprint Resistor_SMD:R_0402_1005Metric -> Package_DFN_QFN:Texas_RJE0020A_VQFN-20-1EP_3x3mm_P0.45mm_EP0.675x0.76mm; symbol Device:R -> Regulator_Switching:TPS568230
- renumbered C40 to C41, C41 to C42, C42 to C43, C45 to C46
Connections:
- net +3V3: now also C40.1, L20.2, R21.1; no longer J1.1, R21.2, R22.1
- net +5V: now also J1.77 (5V), J1.79 (5V), J1.81 (5V), J1.83 (5V), J1.85 (5V), J1.87 (5V), U20.2 (VIN), U20.3 (VIN), U20.4 (VIN), U20.5 (VIN), C45.1, C50.1, C51.1; no longer C48.1, R18.1
- net BST3: now also C49.1, U20.1 (BST); no longer L20.1
- net FB3: now also R21.2, R22.1, U20.14 (FB); no longer C40.1, R22.2
- net GND: now also J1.1 (GND), J1.13 (GND), J1.14 (GND), J1.2 (GND), J1.22 (GND), J1.23 (GND), J1.32 (GND), J1.33 (GND), J1.42 (GND), J1.43 (GND), J1.52 (GND), J1.53 (GND), J1.59 (GND), J1.60 (GND), J1.65 (GND), J1.66 (GND), J1.7 (GND), J1.71 (GND), J1.74 (GND), J1.8 (GND), J1.98 (GND), R22.2, R24.2, U20.13 (AGND), U20.18 (GND), U20.21 (GND), U20.7 (GND), U20.8 (GND), BT50.2 (-), C45.2, C50.2, C51.2, J2.13 (GND), J2.14 (GND), J2.19 (GND), J2.20 (GND), J2.25 (GND), J2.26 (GND), J2.31 (GND), J2.32 (GND), J2.37 (GND), J2.38 (GND), J2.44 (GND), J2.50 (GND), J2.55 (GND), J2.56 (GND), J2.61 (GND), J2.62 (GND), J2.67 (GND), J2.68 (GND), J2.7 (GND), J2.73 (GND), J2.74 (GND), J2.79 (GND), J2.8 (GND), J2.80 (GND), J2.85 (GND), J2.86 (GND), J2.91 (GND), J2.92 (GND), J2.97 (GND), J2.98 (GND), SW50.2, SW51.2; no longer C49.2, R23.2, R25.2, U20.2
- net MODE3: now also R23.2, R24.1, U20.15 (MODE); no longer C49.1, R24.2
- net PG_3V3: now also R25.2, U20.9 (PGOOD); no longer J1.2
- net PG_5V: now also U20.12 (EN); no longer U20.1
- net SW3: now also C49.2, L20.1, U20.19 (SW), U20.20 (SW), U20.6 (SW); no longer L20.2, R21.1
- net VCC3: now also C48.1, U20.17 (VCC); no longer R24.1
- new net: U20.10 (NC), U20.16 (NC)
- new net CM5_1V8: J1.88 (CM5_1.8V), J1.90 (CM5_1.8V)
- new net CM5_3V3: D50.2 (A), D51.2 (A), J1.78 (GPIO_VREF), J1.84 (CM5_3.3V), J1.86 (CM5_3.3V), R18.1
- new net LED_ACT_K: D51.1 (K), R51.1
- new net LED_PWR_K: D50.1 (K), R50.1
- new net LED_nACT: J1.21 (LED_nACT), R51.2
- new net LED_nPWR: J1.95 (LED_nPWR), R50.2
- new net PWR_BUT: J1.92 (PWR_Button), SW50.1
- new net VBAT: BT50.1 (+), J1.76 (VBAT)
- new net nRPIBOOT: J1.93 (nRPIBOOT), SW51.1
- no-connect marks 5 -> 138
Other:
- moved on the sheet: C41, C42, C43, C46, C47, C48, R24

Commit message: cm5: native Gigabit Ethernet port (HR911130A MagJack, TPD4EUSB30 ESD) and its footprint
Follows the official CM5 IO board: pairs 0-3 through two flow-through
TPD4EUSB30 to the MagJack, chip-side centre tap decoupled, activity and
speed LEDs on nLED3/nLED2 through 470R.

hr911130a_fp.py builds the HR911130A footprint from the datasheet
mounting pattern. The LED pin spacing is drawn off scale; the dimensioned
13.25 mm is used and checked against KiCad's HR911105A of the same
housing (--compare). ERC 0, netlist 409/409, review 0 errors.
Parts:
- added C60: 100nF, Capacitor_SMD:C_0402_1005Metric, symbol Device:C
- added J30: HR911130A, CM5:RJ45_Hanrun_HR911130A_Horizontal, symbol CM5_Parts:HR911130A
- added R60, R61: 470, Resistor_SMD:R_0402_1005Metric, symbol Device:R
- added U30, U31: TPD4EUSB30, Package_SON:USON-10_2.5x1.0mm_P0.5mm, symbol Power_Protection:TPD4EUSB30
Connections:
- net CM5_3V3: now also J30.11 (LEDG_A), J30.14 (LEDY_A)
- net GND: now also C60.2, J30.10 (CHS), J30.SH (SHIELD), U30.3 (GND), U30.8 (GND), U31.3 (GND), U31.8 (GND)
- net ETH0_N: now reaches J1.10 (Ethernet_Pair0_N)
- net ETH0_N: now also J30.3 (MDI0-), U30.4 (D2+), U30.7 (NC)
- net ETH2_P: now reaches J1.11 (Ethernet_Pair2_P)
- net ETH2_P: now also J30.5 (MDI2+), U31.5 (D2-), U31.6 (NC)
- net ETH0_P: now reaches J1.12 (Ethernet_Pair0_P)
- net ETH0_P: now also J30.2 (MDI0+), U30.5 (D2-), U30.6 (NC)
- net ETH_nACT: now reaches J1.15 (Ethernet_nLED3)
- net ETH_nACT: now also R60.2
- net ETH_nSPD: now reaches J1.17 (Ethernet_nLED2)
- net ETH_nSPD: now also R61.2
- net ETH3_P: now reaches J1.3 (Ethernet_Pair3_P)
- net ETH3_P: now also J30.8 (MDI3+), U31.1 (D1+), U31.10 (NC)
- net ETH1_P: now reaches J1.4 (Ethernet_Pair1_P)
- net ETH1_P: now also J30.4 (MDI1+), U30.1 (D1+), U30.10 (NC)
- net ETH3_N: now reaches J1.5 (Ethernet_Pair3_N)
- net ETH3_N: now also J30.9 (MDI3-), U31.2 (D1-), U31.9 (NC)
- net ETH1_N: now reaches J1.6 (Ethernet_Pair1_N)
- net ETH1_N: now also J30.7 (MDI1-), U30.2 (D1-), U30.9 (NC)
- net ETH2_N: now reaches J1.9 (Ethernet_Pair2_N)
- net ETH2_N: now also J30.6 (MDI2-), U31.4 (D2+), U31.7 (NC)
- new net ETH_CT: C60.1, J30.1 (CT)
- new net ETH_LEDG_K: J30.12 (LEDG_K), R60.1
- new net ETH_LEDY_K: J30.13 (LEDY_K), R61.1
- no-connect marks 138 -> 128

Commit message: cm5: two LAN7800 USB3-to-Gigabit bridges on USB3-0/USB3-1
Supplies, bias resistors, 25 MHz crystal and USB3 TX coupling caps per
the LAN7800 datasheet (DS00001992H); MAC in OTP, no EEPROM; reset held
by the 3.3 V power-good. MDI pins are no-connect until the PoE block.
The LAN7800 symbol matches datasheet figure 3-1 48/48. review.py knows
the LAN7800 supply ranges and internal regulators; three new mutations
(1.2 V/2.5 V swapped, 3.3 V pin on 5 V) are caught. ERC 0, review 0
errors.
Parts:
- added C100, C110, C130, C140: 10uF, Capacitor_SMD:C_0805_2012Metric, symbol Device:C
- added C101, C102, C103, C104, C106, C107, C108, C109, C111, C112, C113, C114, C115, C120, C121, C131, C132, C133, C134, C136, C137, C138, C139, C141, C142, C143, C144, C145, C150, C151: 100nF, Capacitor_SMD:C_0402_1005Metric, symbol Device:C
- added C105, C117, C135, C147: 1uF, Capacitor_SMD:C_0402_1005Metric, symbol Device:C
- added C118, C119, C148, C149: 27pF, Capacitor_SMD:C_0402_1005Metric, symbol Device:C
- added D40, D42: GREEN, LED_SMD:LED_0805_2012Metric, symbol Device:LED
- added D41, D43: YELLOW, LED_SMD:LED_0805_2012Metric, symbol Device:LED
- added L40, L41: 3.3uH, Inductor_SMD:L_1008_2520Metric, symbol Device:L
- added R100, R130: 2k, Resistor_SMD:R_0402_1005Metric, symbol Device:R
- added R101, R131: 12k, Resistor_SMD:R_0402_1005Metric, symbol Device:R
- added R102, R103, R132, R133: 10k, Resistor_SMD:R_0402_1005Metric, symbol Device:R
- added R104, R105, R134, R135: 470, Resistor_SMD:R_0402_1005Metric, symbol Device:R
- added U40, U41: LAN7800/Y9X, Package_DFN_QFN:QFN-48-1EP_7x7mm_P0.5mm_EP5.3x5.3mm, symbol CM5_Parts:LAN7800
- added Y40, Y41: 25MHz, Crystal:Crystal_SMD_3225-4Pin_3.2x2.5mm, symbol Device:Crystal_GND24
Connections:
- net +3V3: now also C100.1, C101.1, C102.1, C103.1, C104.1, C130.1, C131.1, C132.1, C133.1, C134.1, D40.2 (A), D41.2 (A), D42.2 (A), D43.2 (A), U40.14 (VDD_SW_IN), U40.20 (VDDVARIO), U40.23 (VBUS_DET), U40.36 (VDDVARIO), U40.38 (VDD33A), U40.39 (VDDVARIO), U40.46 (VDD33_REG_IN), U41.14 (VDD_SW_IN), U41.20 (VDDVARIO), U41.23 (VBUS_DET), U41.36 (VDDVARIO), U41.38 (VDD33A), U41.39 (VDDVARIO), U41.46 (VDD33_REG_IN)
- net GND: now also C100.2, C101.2, C102.2, C103.2, C104.2, C105.2, C106.2, C107.2, C108.2, C109.2, C110.2, C111.2, C112.2, C113.2, C114.2, C115.2, C117.2, C118.2, C119.2, C130.2, C131.2, C132.2, C133.2, C134.2, C135.2, C136.2, C137.2, C138.2, C139.2, C140.2, C141.2, C142.2, C143.2, C144.2, C145.2, C147.2, C148.2, C149.2, R100.2, R101.2, R102.2, R103.2, R130.2, R131.2, R132.2, R133.2, U40.34 (TEST), U40.49 (VSS), U41.34 (TEST), U41.49 (VSS), Y40.2 (G), Y40.4 (G), Y41.2 (G), Y41.4 (G)
- net PG_3V3: now also U40.35 (RESET_N/PME_CLEAR), U41.35 (RESET_N/PME_CLEAR)
- net CM5U0_RX_N: now reaches J2.28 (USB3-0-RX_N)
- net CM5U0_RX_N: now also C121.2
- net CM5U0_RX_P: now reaches J2.30 (USB3-0-RX_P)
- net CM5U0_RX_P: now also C120.2
- net LAN0_DP: now reaches J2.34 (USB3-0-DP)
- net LAN0_DP: now also U40.26 (USB2_DP)
- net LAN0_DM: now reaches J2.36 (USB3-0-DM)
- net LAN0_DM: now also U40.27 (USB2_DM)
- net LAN0_RX_N: now reaches J2.40 (USB3-0-TX_N)
- net LAN0_RX_N: now also U40.32 (USB3_RXDM)
- net LAN0_RX_P: now reaches J2.42 (USB3-0-TX_P)
- net LAN0_RX_P: now also U40.31 (USB3_RXDP)
- net CM5U1_RX_N: now reaches J2.57 (USB3-1-RX_N)
- net CM5U1_RX_N: now also C151.2
- net CM5U1_RX_P: now reaches J2.59 (USB3-1-RX_P)
- net CM5U1_RX_P: now also C150.2
- net LAN1_DP: now reaches J2.63 (USB3-1-DP)
- net LAN1_DP: now also U41.26 (USB2_DP)
- net LAN1_DM: now reaches J2.65 (USB3-1-DM)
- net LAN1_DM: now also U41.27 (USB2_DM)
- net LAN1_RX_N: now reaches J2.69 (USB3-1-TX_N)
- net LAN1_RX_N: now also U41.32 (USB3_RXDM)
- net LAN1_RX_P: now reaches J2.71 (USB3-1-TX_P)
- net LAN1_RX_P: now also U41.31 (USB3_RXDP)
- new net LAN0_1V2: C110.1, C111.1, C112.1, C113.1, C114.1, C115.1, L40.2, U40.15 (VDD12_SW_FB), U40.21 (VDD12CORE), U40.25 (VDD12A), U40.30 (VDD12A), U40.42 (VDD12CORE), U40.44 (VDD12A)
- new net LAN0_2V5: C105.1, C106.1, C107.1, C108.1, C109.1, U40.12 (VDD25A), U40.3 (VDD25A), U40.45 (VDD25_REG_OUT), U40.6 (VDD25A), U40.9 (VDD25A)
- new net LAN0_EEDI: R102.1, U40.17 (EEDI/GPIO1)
- new net LAN0_FILT: C117.1, U40.48 (REF_FILT)
- new net LAN0_LEDG_K: R104.2, U40.18 (EEDO/LED0/GPIO2)
- new net LAN0_LEDG_K2: D40.1 (K), R104.1
- new net LAN0_LEDY_K: R105.2, U40.19 (EECLK/LED1/GPIO3)
- new net LAN0_LEDY_K2: D41.1 (K), R105.1
- new net LAN0_PMEMODE: R103.1, U40.43 (PME_MODE/GPIO7)
- new net LAN0_RBIAS: R101.1, U40.37 (USBRBIAS)
- new net LAN0_REXT: R100.1, U40.47 (REF_REXT)
- new net LAN0_SW: L40.1, U40.13 (VDD12_SW_OUT)
- new net LAN0_TX_N: C121.1, U40.29 (USB3_TXDM)
- new net LAN0_TX_P: C120.1, U40.28 (USB3_TXDP)
- new net LAN0_XI: C118.1, U40.40 (XI), Y40.1
- new net LAN0_XO: C119.1, U40.41 (XO), Y40.3
- new net LAN1_1V2: C140.1, C141.1, C142.1, C143.1, C144.1, C145.1, L41.2, U41.15 (VDD12_SW_FB), U41.21 (VDD12CORE), U41.25 (VDD12A), U41.30 (VDD12A), U41.42 (VDD12CORE), U41.44 (VDD12A)
- new net LAN1_2V5: C135.1, C136.1, C137.1, C138.1, C139.1, U41.12 (VDD25A), U41.3 (VDD25A), U41.45 (VDD25_REG_OUT), U41.6 (VDD25A), U41.9 (VDD25A)
- new net LAN1_EEDI: R132.1, U41.17 (EEDI/GPIO1)
- new net LAN1_FILT: C147.1, U41.48 (REF_FILT)
- new net LAN1_LEDG_K: R134.2, U41.18 (EEDO/LED0/GPIO2)
- new net LAN1_LEDG_K2: D42.1 (K), R134.1
- new net LAN1_LEDY_K: R135.2, U41.19 (EECLK/LED1/GPIO3)
- new net LAN1_LEDY_K2: D43.1 (K), R135.1
- new net LAN1_PMEMODE: R133.1, U41.43 (PME_MODE/GPIO7)
- new net LAN1_RBIAS: R131.1, U41.37 (USBRBIAS)
- new net LAN1_REXT: R130.1, U41.47 (REF_REXT)
- new net LAN1_SW: L41.1, U41.13 (VDD12_SW_OUT)
- new net LAN1_TX_N: C151.1, U41.29 (USB3_TXDM)
- new net LAN1_TX_P: C150.1, U41.28 (USB3_TXDP)
- new net LAN1_XI: C148.1, U41.40 (XI), Y41.1
- new net LAN1_XO: C149.1, U41.41 (XO), Y41.3
- no-connect marks 128 -> 140

Commit message: cm5: two 802.3at PoE ports (IP804AR PSE, G2423S magnetics, RJHSE5380) on the LAN7800s
IP804AR in auto mode without EEPROM, ports 0/1, Alternative A. G2423S
footprint generated from the datasheet land pattern; IP804AR symbol
matches the datasheet pin table 48/48. rails.json declares the 54 V
input range so review.py can check V54 against 802.3at (50-57 V); two
new mutations are caught.

netlabel: no NC flag on pins whose electrical type is already
no_connect (KiCad reported one as dangling). relay8 loses one redundant
flag; its ERC and netlist are unchanged.
Parts:
- added C70, C71, C72, C73, C74, C75, C76, C77, C88: 100nF, Capacitor_SMD:C_0402_1005Metric, symbol Device:C
- added C82: 1uF, Capacitor_SMD:C_1206_3216Metric, symbol Device:C
- added C83: 47uF, Capacitor_SMD:CP_Elec_10x10, symbol Device:C_Polarized
- added C84, C85, C86, C87: 4.7uF, Capacitor_SMD:C_0603_1608Metric, symbol Device:C
- added C90, C91: 1nF 2kV, Capacitor_SMD:C_1206_3216Metric, symbol Device:C
- added C92, C93: 100nF, Capacitor_SMD:C_0805_2012Metric, symbol Device:C
- added D60, D61: SM6T68A, Diode_SMD:D_SMB, symbol Diode:SM6T68A
- added F40, F41: 1.5A, Fuse:Fuse_1206_3216Metric, symbol Device:Fuse
- added J40: POE0, Connector_RJ:RJ45_Amphenol_RJHSE5380, symbol Connector:RJ45_Shielded
- added J41: POE1, Connector_RJ:RJ45_Amphenol_RJHSE5380, symbol Connector:RJ45_Shielded
- added R74, R75, R76, R77, R78: 10k, Resistor_SMD:R_0402_1005Metric, symbol Device:R
- added R80, R81, R82, R83: 75, Resistor_SMD:R_0603_1608Metric, symbol Device:R
- added T40, T41: G2423S, CM5:Transformer_CNDtek_G2423S, symbol CM5_Parts:G2423S
- added U50: IP804AR, Package_DFN_QFN:QFN-48-1EP_7x7mm_P0.5mm_EP5.3x5.3mm, symbol CM5_Parts:IP804AR
Connections:
- net +54V: now also C82.1, C83.1, F40.1, F41.1, U50.17 (V54)
- net GND: now also C70.2, C71.2, C72.2, C73.2, C74.2, C75.2, C76.2, C77.2, C82.2, C83.2, C84.2, C85.2, C86.2, C87.2, C88.2, C90.2, C91.2, J40.SH, J41.SH, R77.2, R78.2, U50.1 (AGND), U50.11 (AGND), U50.12 (AGND), U50.13 (SCAN0), U50.14 (SCAN1), U50.23 (In_Top), U50.24 (EnB_Reg), U50.25 (AGND), U50.26 (AGND), U50.27 (AGND), U50.28 (ALT_A/B), U50.29 (24V_En), U50.30 (4Pair_En), U50.31 (AGND), U50.43 (DGND), U50.46 (AD2), U50.47 (AD1), U50.48 (AD0), U50.49 (EPAD), U50.6 (AGND)
- net LAN0_TR0P: now reaches U40.1 (TR0P)
- net LAN0_TR0P: now also T40.23 (TD1+)
- net LAN0_TR3P: now reaches U40.10 (TR3P)
- net LAN0_TR3P: now also T40.14 (TD4+)
- net LAN0_TR3N: now reaches U40.11 (TR3N)
- net LAN0_TR3N: now also T40.13 (TD4-)
- net LAN0_TR0N: now reaches U40.2 (TR0N)
- net LAN0_TR0N: now also T40.22 (TD1-)
- net LAN0_TR1P: now reaches U40.4 (TR1P)
- net LAN0_TR1P: now also T40.20 (TD2+)
- net LAN0_TR1N: now reaches U40.5 (TR1N)
- net LAN0_TR1N: now also T40.19 (TD2-)
- net LAN0_TR2P: now reaches U40.7 (TR2P)
- net LAN0_TR2P: now also T40.17 (TD3+)
- net LAN0_TR2N: now reaches U40.8 (TR2N)
- net LAN0_TR2N: now also T40.16 (TD3-)
- net LAN1_TR0P: now reaches U41.1 (TR0P)
- net LAN1_TR0P: now also T41.23 (TD1+)
- net LAN1_TR3P: now reaches U41.10 (TR3P)
- net LAN1_TR3P: now also T41.14 (TD4+)
- net LAN1_TR3N: now reaches U41.11 (TR3N)
- net LAN1_TR3N: now also T41.13 (TD4-)
- net LAN1_TR0N: now reaches U41.2 (TR0N)
- net LAN1_TR0N: now also T41.22 (TD1-)
- net LAN1_TR1P: now reaches U41.4 (TR1P)
- net LAN1_TR1P: now also T41.20 (TD2+)
- net LAN1_TR1N: now reaches U41.5 (TR1N)
- net LAN1_TR1N: now also T41.19 (TD2-)
- net LAN1_TR2P: now reaches U41.7 (TR2P)
- net LAN1_TR2P: now also T41.17 (TD3+)
- net LAN1_TR2N: now reaches U41.8 (TR2N)
- net LAN1_TR2N: now also T41.16 (TD3-)
- new net IP_1V8: C87.1, U50.21 (V1P8)
- new net IP_3V3: C85.1, C86.1, R74.1, R75.1, R76.1, U50.20 (V3P3), U50.44 (DV3P3)
- new net IP_5V: C84.1, U50.19 (V5), U50.22 (VPP)
- new net IP_LEDCLK: R77.1, U50.37 (LED_CLK)
- new net IP_LEDDAT: R78.1, U50.38 (LED_DAT)
- new net IP_RSTN: C88.1, R74.2, U50.45 (RstN)
- new net IP_SCL: R75.2, U50.39 (SCL/EE_CLK)
- new net IP_SDA: R76.2, U50.41 (SDAI/EE_DAT)
- new net POE0_A_N: J40.2, T40.3 (MX1-)
- new net POE0_A_P: J40.1, T40.2 (MX1+)
- new net POE0_BOB: C90.1, R80.2, R81.2
- new net POE0_B_N: J40.6, T40.6 (MX2-)
- new net POE0_B_P: J40.3, T40.5 (MX2+)
- new net POE0_CT3: R80.1, T40.7 (MCT3)
- new net POE0_CT4: R81.1, T40.10 (MCT4)
- new net POE0_C_N: J40.5, T40.9 (MX3-)
- new net POE0_C_P: J40.4, T40.8 (MX3+)
- new net POE0_D_N: J40.8, T40.12 (MX4-)
- new net POE0_D_P: J40.7, T40.11 (MX4+)
- new net POE0_N: C92.2, D60.2 (A2), T40.1 (MCT1), U50.3 (PortN0)
- new net POE0_P: C92.1, D60.1 (A1), F40.2, T40.4 (MCT2)
- new net POE0_TCT1: C70.1, T40.24 (TCT1)
- new net POE0_TCT2: C71.1, T40.21 (TCT2)
- new net POE0_TCT3: C72.1, T40.18 (TCT3)
- new net POE0_TCT4: C73.1, T40.15 (TCT4)
- new net POE1_A_N: J41.2, T41.3 (MX1-)
- new net POE1_A_P: J41.1, T41.2 (MX1+)
- new net POE1_BOB: C91.1, R82.2, R83.2
- new net POE1_B_N: J41.6, T41.6 (MX2-)
- new net POE1_B_P: J41.3, T41.5 (MX2+)
- new net POE1_CT3: R82.1, T41.7 (MCT3)
- new net POE1_CT4: R83.1, T41.10 (MCT4)
- new net POE1_C_N: J41.5, T41.9 (MX3-)
- new net POE1_C_P: J41.4, T41.8 (MX3+)
- new net POE1_D_N: J41.8, T41.12 (MX4-)
- new net POE1_D_P: J41.7, T41.11 (MX4+)
- new net POE1_N: C93.2, D61.2 (A2), T41.1 (MCT1), U50.5 (PortN1)
- new net POE1_P: C93.1, D61.1 (A1), F41.2, T41.4 (MCT2)
- new net POE1_TCT1: C74.1, T41.24 (TCT1)
- new net POE1_TCT2: C75.1, T41.21 (TCT2)
- new net POE1_TCT3: C76.1, T41.18 (TCT3)
- new net POE1_TCT4: C77.1, T41.15 (TCT4)
- no-connect marks 140 -> 131
