File: boards/cm5/cm5.kicad_sch (KiCad schematic)
At the start: 171 parts, among them J1 CM5 pins 1-100, J2 CM5 pins 101-200, J20 54V IN, J30 HR911130A, J40 POE0, J41 POE1, Q10 BSC160N10NS3G, Q11 BSC070N10NS5, SW50 POWER, SW51 RPIBOOT, T40 G2423S, T41 G2423S, U10 LM5146RGYR, U20 TPS568230RJER, U30 TPD4EUSB30, U31 TPD4EUSB30, U40 LAN7800/Y9X, U41 LAN7800/Y9X, U50 IP804AR, Y40 25MHz, Y41 25MHz

Commit message: cm5: USB 2.0 block (FSUSB42 switch, USB2514B hub with two USB-A ports, USB-C flashing port)
A single slide switch replaces the rpiboot button: FLASH holds nRPIBOOT
low and leaves USB_OTG_ID floating (device), RUN grounds USB_OTG_ID
(host). The FSUSB42 select follows nRPIBOOT and is powered from
CM5_3V3, the same domain. Hub in default configuration with ports 3/4
disabled, AP2171W per-port power switches, USBLC6 on every connector.
review.py knows the USB2514B and FSUSB42 supply ranges and treats USB-A
VBUS as a valid ESD reference; three new mutations are caught. ERC 0,
netlist 977/977, review 0 errors.
Parts:
- added C200, C202, C203, C204, C205, C206, C207, C212, C215: 100nF, Capacitor_SMD:C_0402_1005Metric, symbol Device:C
- added C201: 4.7uF, Capacitor_SMD:C_0603_1608Metric, symbol Device:C
- added C208, C209: 27pF, Capacitor_SMD:C_0402_1005Metric, symbol Device:C
- added C210, C213: 1uF, Capacitor_SMD:C_0402_1005Metric, symbol Device:C
- added C211, C214: 100uF, Capacitor_SMD:CP_Elec_6.3x7.7, symbol Device:C_Polarized
- added D70, D71, D72: USBLC6-2SC6, Package_TO_SOT_SMD:SOT-23-6, symbol Power_Protection:USBLC6-2SC6
- added J50: USB-C FLASH, Connector_USB:USB_C_Receptacle_HRO_TYPE-C-31-M-12, symbol Connector:USB_C_Receptacle_USB2.0_16P
- added J51: USB-A 1, Connector_USB:USB_A_Molex_48037-2200_Horizontal, symbol Connector:USB_A
- added J52: USB-A 2, Connector_USB:USB_A_Molex_48037-2200_Horizontal, symbol Connector:USB_A
- added R200, R201: 5.1k, Resistor_SMD:R_0402_1005Metric, symbol Device:R
- added R202, R203, R204: 100k, Resistor_SMD:R_0402_1005Metric, symbol Device:R
- added R205, R206, R207, R208, R209: 10k, Resistor_SMD:R_0402_1005Metric, symbol Device:R
- added R210: 12k, Resistor_SMD:R_0402_1005Metric, symbol Device:R
- added R211: 1M, Resistor_SMD:R_0402_1005Metric, symbol Device:R
- added U60: FSUSB42MUX, Package_SO:MSOP-10_3x3mm_P0.5mm, symbol Interface_USB:FSUSB42MUX
- added U61: USB2514B, Package_DFN_QFN:QFN-36-1EP_6x6mm_P0.5mm_EP3.7x3.7mm, symbol Interface_USB:USB2514B_Bi
- added U62, U63: AP2171W, Package_TO_SOT_SMD:SOT-23-5, symbol Power_Management:AP2171W
- added Y60: 24MHz, Crystal:Crystal_SMD_3225-4Pin_3.2x2.5mm, symbol Device:Crystal_GND24
- SW51: value RPIBOOT -> FLASH/RUN; footprint Button_Switch_SMD:SW_Push_1P1T_NO_CK_KMR2 -> Button_Switch_SMD:SW_SPDT_PCM12; symbol Switch:SW_Push -> Switch:SW_SPDT
Connections:
- net +3V3: now also C201.1, C202.1, C203.1, C204.1, C205.1, R205.1, R206.1, R207.1, R208.1, R209.1, U61.10 (VDDA33), U61.15 (VDD33), U61.23 (VDD33), U61.27 (VBUS_DET), U61.29 (VDDA33), U61.36 (VDDA33), U61.5 (VDDA33)
- net +5V: now also C210.1, C213.1, U62.5 (IN), U63.5 (IN)
- net CM5_3V3: now also C200.1, U60.1 (VCC)
- net GND: now also C200.2, C201.2, C202.2, C203.2, C204.2, C205.2, C206.2, C207.2, C208.2, C209.2, C210.2, C211.2, C212.2, C213.2, C214.2, C215.2, D70.2 (GND), D71.2 (GND), D72.2 (GND), J50.A1 (GND), J50.A12 (GND), J50.B1 (GND), J50.B12 (GND), J50.SH (SHIELD), J51.4 (GND), J51.SH (Shield), J52.4 (GND), J52.SH (Shield), R200.2, R201.2, R202.2, R203.2, R204.2, R210.2, U60.10 (~{OE}), U60.5 (GND), U61.11 (TEST), U61.37 (VSS), U62.2 (GND), U63.2 (GND), Y60.2 (G), Y60.4 (G)
- net PG_3V3: now also U61.26 (RESET_N)
- net nRPIBOOT: now also U60.2 (SEL)
- net USB_OTG_ID: now reaches J2.1 (USB_OTG_ID)
- net USB_OTG_ID: now also SW51.3 (C)
- net CM5_USB_N: now reaches J2.3 (USB_N)
- net CM5_USB_N: now also U60.4 (D-)
- net CM5_USB_P: now reaches J2.5 (USB_P)
- net CM5_USB_P: now also U60.3 (D+)
- new net HUB_CFG0: R202.1, U61.24 (SCL/SMBCLK/CFG_SEL0)
- new net HUB_CFG1: R203.1, U61.25 (HS_IND/CFG_SEL1)
- new net HUB_CRFILT: C206.1, U61.14 (CRFILT)
- new net HUB_DIS3: R205.2, U61.6 (USBDM_DN3/PRT_DIS_M3), U61.7 (USBDP_DN3/PRT_DIS_P3)
- new net HUB_DIS4: R206.2, U61.8 (USBDM_DN4/PRT_DIS_M4), U61.9 (USBDP_DN4/PRT_DIS_P4)
- new net HUB_NONREM1: R204.1, U61.22 (SDA/SMBDATA/NON_REM1)
- new net HUB_OCN34: R207.2, U61.19 (OCS_N3), U61.21 (OCS_N4)
- new net HUB_PLLFILT: C207.1, U61.34 (PLLFILT)
- new net HUB_RBIAS: R210.1, U61.35 (RBIAS)
- new net HUB_UP_DN: U60.8 (HSD2-), U61.30 (USBDM_UP)
- new net HUB_UP_DP: U60.9 (HSD2+), U61.31 (USBDP_UP)
- new net HUB_XI: C208.1, R211.1, U61.33 (XTALIN/CLKIN), Y60.1
- new net HUB_XO: C209.1, R211.2, U61.32 (XTALOUT), Y60.3
- new net USBA0_DN: D71.3 (I/O2), D71.4 (I/O2), J51.2 (D-), U61.1 (USBDM_DN1/PRT_DIS_M1)
- new net USBA0_DP: D71.1 (I/O1), D71.6 (I/O1), J51.3 (D+), U61.2 (USBDP_DN1/PRT_DIS_P1)
- new net USBA0_EN: U61.12 (PRTPWR1/BC_EN1), U62.4 (EN)
- new net USBA0_OCN: R208.2, U61.13 (OCS_N1), U62.3 (~{FLG})
- new net USBA0_VBUS: C211.1, C212.1, D71.5 (VBUS), J51.1 (VBUS), U62.1 (OUT)
- new net USBA1_DN: D72.3 (I/O2), D72.4 (I/O2), J52.2 (D-), U61.3 (USBDM_DN2/PRT_DIS_M2)
- new net USBA1_DP: D72.1 (I/O1), D72.6 (I/O1), J52.3 (D+), U61.4 (USBDP_DN2/PRT_DIS_P2)
- new net USBA1_EN: U61.16 (PRTPWR2/BC_EN2), U63.4 (EN)
- new net USBA1_OCN: R209.2, U61.17 (OCS_N2), U63.3 (~{FLG})
- new net USBA1_VBUS: C214.1, C215.1, D72.5 (VBUS), J52.1 (VBUS), U63.1 (OUT)
- new net USBC_CC1: J50.A5 (CC1), R200.1
- new net USBC_CC2: J50.B5 (CC2), R201.1
- new net USBC_DN: D70.3 (I/O2), D70.4 (I/O2), J50.A7 (D-), J50.B7 (D-), U60.6 (HSD1-)
- new net USBC_DP: D70.1 (I/O1), D70.6 (I/O1), J50.A6 (D+), J50.B6 (D+), U60.7 (HSD1+)
- new net USBC_VBUS: D70.5 (VBUS), J50.A4 (VBUS), J50.A9 (VBUS), J50.B4 (VBUS), J50.B9 (VBUS)
- no-connect marks 131 -> 133

Commit message: cm5: M.2 M-key socket for PCIe NVMe, with a generated TE 1-2199230-6 footprint
Pinout follows the official CM5 IO board; 3.3 V comes straight from
+3V3. m2_fp.py builds the socket footprint (with 2230-2280 standoff
holes) from TE drawing C-2199230 and matches the official footprint
67/67 pads. Note 2199230-4 without the 1- prefix is the E-key part.
review.py checks the M.2 3.3 V pins (+/-5 %); new mutation caught.
Sheet is A0. ERC 0, netlist 1050/1050, review 0 errors.
Parts:
- added C220, C221: 47uF, Capacitor_SMD:C_1210_3225Metric, symbol Device:C
- added C222: 100nF, Capacitor_SMD:C_0402_1005Metric, symbol Device:C
- added J60: M.2 M-key, CM5:M.2_Socket_M_TE_1-2199230-6, symbol Connector:Bus_M.2_Socket_M
Connections:
- net +3V3: now also C220.1, C221.1, C222.1, J60.12 (3.3V), J60.14 (3.3V), J60.16 (3.3V), J60.18 (3.3V), J60.2 (3.3V), J60.4 (3.3V), J60.70 (3.3V), J60.72 (3.3V), J60.74 (3.3V)
- net GND: now also C220.2, C221.2, C222.2, J60.1 (GND), J60.15 (GND), J60.21 (GND), J60.27 (GND), J60.3 (GND), J60.33 (GND), J60.39 (GND), J60.45 (GND), J60.51 (GND), J60.57 (GND), J60.71 (GND), J60.73 (GND), J60.75 (GND), J60.9 (GND)
- net PCIE_CLK_P: now reaches J2.10 (PCIe_CLK_P)
- net PCIE_CLK_P: now also J60.55 (REFCLKp)
- net PCIE_CLK_N: now reaches J2.12 (PCIe_CLK_N)
- net PCIE_CLK_N: now also J60.53 (REFCLKn)
- net PCIE_RX_P: now reaches J2.16 (PCIe_RX_P)
- net PCIE_RX_P: now also J60.41 (PERn0/SATA-B+)
- net PCIE_RX_N: now reaches J2.18 (PCIe_RX_N)
- net PCIE_RX_N: now also J60.43 (PERp0/SATA-B-)
- net PCIE_nCLKREQ: now reaches J2.2 (PCIe_CLK_nREQ)
- net PCIE_nCLKREQ: now also J60.52 (~{CLKREQ})
- net PCIE_TX_P: now reaches J2.22 (PCIe_TX_P)
- net PCIE_TX_P: now also J60.47 (PETn0/SATA-A-)
- net PCIE_TX_N: now reaches J2.24 (PCIe_TX_N)
- net PCIE_TX_N: now also J60.49 (PETp0/SATA-A+)
- net PCIE_nWAKE: now reaches J2.4 (PCIE_nWAKE)
- net PCIE_nWAKE: now also J60.54 (~{PEWAKE})
- net PCIE_nRST: now reaches J2.9 (PCIe_nRST)
- net PCIE_nRST: now also J60.50 (~{PERST})
- no-connect marks 133 -> 140

Commit message: cm5: HDMI0 port (Molex 208658-1001) with a TPS2051C-limited 5 V enabled by CM5_3V3
TMDS, DDC, CEC and HPD wired as on the official CM5 IO board. ERC 0,
netlist 1079/1079, review 0 errors.
Parts:
- added C230, C231: 100nF, Capacitor_SMD:C_0402_1005Metric, symbol Device:C
- added J70: HDMI, Connector_Video:HDMI_A_Molex_208658-1001_Horizontal, symbol Connector:HDMI_A
- added U70: TPS2051CDBV, Package_TO_SOT_SMD:SOT-23-5, symbol Power_Management:TPS2051CDBV
Connections:
- net +5V: now also C230.1, U70.5 (IN)
- net CM5_3V3: now also U70.4 (EN)
- net GND: now also C230.2, C231.2, J70.11 (CKS), J70.17 (GND), J70.2 (D2S), J70.5 (D1S), J70.8 (D0S), J70.SH, U70.2 (GND)
- net HDMI0_SCL: now reaches J2.100 (HDMI0_SCL)
- net HDMI0_SCL: now also J70.15 (SCL)
- net HDMI0_CEC: now reaches J2.51 (HDMI0_CEC)
- net HDMI0_CEC: now also J70.13 (CEC)
- net HDMI0_HPD: now reaches J2.53 (HDMI0_HOTPLUG)
- net HDMI0_HPD: now also J70.19 (HPD)
- net HDMI0_D2_P: now reaches J2.70 (HDMI0_TX2_P)
- net HDMI0_D2_P: now also J70.1 (D2+)
- net HDMI0_D2_N: now reaches J2.72 (HDMI0_TX2_N)
- net HDMI0_D2_N: now also J70.3 (D2-)
- net HDMI0_D1_P: now reaches J2.76 (HDMI0_TX1_P)
- net HDMI0_D1_P: now also J70.4 (D1+)
- net HDMI0_D1_N: now reaches J2.78 (HDMI0_TX1_N)
- net HDMI0_D1_N: now also J70.6 (D1-)
- net HDMI0_D0_P: now reaches J2.82 (HDMI0_TX0_P)
- net HDMI0_D0_P: now also J70.7 (D0+)
- net HDMI0_D0_N: now reaches J2.84 (HDMI0_TX0_N)
- net HDMI0_D0_N: now also J70.9 (D0-)
- net HDMI0_CK_P: now reaches J2.88 (HDMI0_CLK_P)
- net HDMI0_CK_P: now also J70.10 (CK+)
- net HDMI0_CK_N: now reaches J2.90 (HDMI0_CLK_N)
- net HDMI0_CK_N: now also J70.12 (CK-)
- net HDMI0_SDA: now reaches J2.99 (HDMI0_SDA)
- net HDMI0_SDA: now also J70.16 (SDA)
- new net HDMI_5V: C231.1, J70.18 (+5V), U70.1 (OUT)
- no-connect marks 140 -> 130
