File: boards/cm5/cm5.kicad_sch (KiCad schematic)
At the start: 218 parts, among them J1 CM5 pins 1-100, J2 CM5 pins 101-200, J20 54V IN, J30 HR911130A, J40 POE0, J41 POE1, J50 USB-C FLASH, J51 USB-A 1, J52 USB-A 2, J60 M.2 M-key, J70 HDMI, Q10 BSC160N10NS3G, Q11 BSC070N10NS5, SW50 POWER, SW51 FLASH/RUN, T40 G2423S, T41 G2423S, U10 LM5146RGYR, U20 TPS568230RJER, U30 TPD4EUSB30, U31 TPD4EUSB30, U40 LAN7800/Y9X, U41 LAN7800/Y9X, U50 IP804AR, U60 FSUSB42MUX, U61 USB2514B, U62 AP2171W, U63 AP2171W, U70 TPS2051CDBV, Y40 25MHz, Y41 25MHz, Y60 24MHz

Commit message: cm5: 40-pin GPIO header and fan connector; schematic complete
GPIO0-27 to a standard 2x20 header (matches the official CM5 IO board J8
pin for pin), fan on a JST SH 4-pin with the Raspberry Pi active cooler
pinout. ERC 0, netlist 1126/1126, review 0 errors.
Parts:
- added J80: GPIO 40-pin, Connector_PinHeader_2.54mm:PinHeader_2x20_P2.54mm_Vertical, symbol Connector_Generic:Conn_02x20_Odd_Even
- added J81: FAN, Connector_JST:JST_SH_SM04B-SRSS-TB_1x04-1MP_P1.00mm_Horizontal, symbol Connector_Generic_MountingPin:Conn_01x04_MountingPin
- added R230: 10k, Resistor_SMD:R_0402_1005Metric, symbol Device:R
Connections:
- net +5V: now also J80.2 (Pin_2), J80.4 (Pin_4), J81.1 (Pin_1)
- net CM5_3V3: now also J80.1 (Pin_1), J80.17 (Pin_17), R230.1
- net GND: now also J80.14 (Pin_14), J80.20 (Pin_20), J80.25 (Pin_25), J80.30 (Pin_30), J80.34 (Pin_34), J80.39 (Pin_39), J80.6 (Pin_6), J80.9 (Pin_9), J81.3 (Pin_3), J81.MP (MountPin)
- net FAN_TACHO: now reaches J1.16 (Fan_Tacho)
- net FAN_TACHO: now also J81.4 (Pin_4)
- net FAN_PWM: now reaches J1.19 (Fan_PWM)
- net FAN_PWM: now also J81.2 (Pin_2), R230.2
- net GPIO26: now reaches J1.24 (GPIO26)
- net GPIO26: now also J80.37 (Pin_37)
- net GPIO21: now reaches J1.25 (GPIO21)
- net GPIO21: now also J80.40 (Pin_40)
- net GPIO19: now reaches J1.26 (GPIO19)
- net GPIO19: now also J80.35 (Pin_35)
- net GPIO20: now reaches J1.27 (GPIO20)
- net GPIO20: now also J80.38 (Pin_38)
- net GPIO13: now reaches J1.28 (GPIO13)
- net GPIO13: now also J80.33 (Pin_33)
- net GPIO16: now reaches J1.29 (GPIO16)
- net GPIO16: now also J80.36 (Pin_36)
- net GPIO6: now reaches J1.30 (GPIO6)
- net GPIO6: now also J80.31 (Pin_31)
- net GPIO12: now reaches J1.31 (GPIO12)
- net GPIO12: now also J80.32 (Pin_32)
- net GPIO5: now reaches J1.34 (GPIO5)
- net GPIO5: now also J80.29 (Pin_29)
- net ID_SC: now reaches J1.35 (ID_SC)
- net ID_SC: now also J80.28 (Pin_28)
- net ID_SD: now reaches J1.36 (ID_SD)
- net ID_SD: now also J80.27 (Pin_27)
- net GPIO7: now reaches J1.37 (GPIO7)
- net GPIO7: now also J80.26 (Pin_26)
- net GPIO11: now reaches J1.38 (GPIO11)
- net GPIO11: now also J80.23 (Pin_23)
- net GPIO8: now reaches J1.39 (GPIO8)
- net GPIO8: now also J80.24 (Pin_24)
- net GPIO9: now reaches J1.40 (GPIO9)
- net GPIO9: now also J80.21 (Pin_21)
- net GPIO25: now reaches J1.41 (GPIO25)
- net GPIO25: now also J80.22 (Pin_22)
- net GPIO10: now reaches J1.44 (GPIO10)
- net GPIO10: now also J80.19 (Pin_19)
- net GPIO24: now reaches J1.45 (GPIO24)
- net GPIO24: now also J80.18 (Pin_18)
- net GPIO22: now reaches J1.46 (GPIO22)
- net GPIO22: now also J80.15 (Pin_15)
- net GPIO23: now reaches J1.47 (GPIO23)
- net GPIO23: now also J80.16 (Pin_16)
- net GPIO27: now reaches J1.48 (GPIO27)
- net GPIO27: now also J80.13 (Pin_13)
- net GPIO18: now reaches J1.49 (GPIO18)
- net GPIO18: now also J80.12 (Pin_12)
- net GPIO17: now reaches J1.50 (GPIO17)
- net GPIO17: now also J80.11 (Pin_11)
- net GPIO15: now reaches J1.51 (GPIO15)
- net GPIO15: now also J80.10 (Pin_10)
- net GPIO4: now reaches J1.54 (GPIO4)
- net GPIO4: now also J80.7 (Pin_7)
- net GPIO14: now reaches J1.55 (GPIO14)
- net GPIO14: now also J80.8 (Pin_8)
- net GPIO3: now reaches J1.56 (GPIO3)
- net GPIO3: now also J80.5 (Pin_5)
- net GPIO2: now reaches J1.58 (GPIO2)
- net GPIO2: now also J80.3 (Pin_3)
- no-connect marks 130 -> 100
