File: boards/cm5/cm5.kicad_pcb (KiCad board)
At the start: 4 copper layers, 170 x 120 mm, 229 parts, among them J1 CM5 pins 1-100, J2 CM5 pins 101-200, J20 54V IN, J30 HR911130A, J40 POE0, J41 POE1, J50 USB-C FLASH, J51 USB-A 1, J52 USB-A 2, J60 M.2 M-key, J70 HDMI, J80 GPIO 40-pin, J81 FAN, Q10 BSC160N10NS3G, Q11 BSC070N10NS5, SW50 POWER, SW51 FLASH/RUN, T40 G2423S, T41 G2423S, U10 LM5146RGYR, U20 TPS568230RJER, U30 TPD4EUSB30, U31 TPD4EUSB30, U40 LAN7800/Y9X, U41 LAN7800/Y9X, U50 IP804AR, U60 FSUSB42MUX, U61 USB2514B, U62 AP2171W, U63 AP2171W, U70 TPS2051CDBV, Y40 25MHz, Y41 25MHz, Y60 24MHz

Commit message: cm5: inner GND plane and split +5V/+3V3 plane with a current check (#17)
L2 is a solid ground plane, the reference for the L1 differential pairs.
L3 is split: +5V top right (buck output to CM5, 40-pin header, fan) and
an L-shaped +3V3 along the bottom and left edges (to the hub, both
LAN7800s and the M.2 socket).

gen/pcb.py checks each current corridor: it must lie inside its net's
plane and be at least as wide as IPC-2221 6.2 asks for on a 0.5 oz inner
layer at a 10 C rise. Failing removes the board file instead of leaving
one without planes. Shrinking the +5V plane or raising its current to
30 A both fail.
Routing:
- added copper zone on In2.Cu, net +3V3
- added copper zone on In2.Cu, net +5V
- added copper zone on In1.Cu, net GND
Changed lines of the file:
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@@
 		(layer "Edge.Cuts")
+	)
+	(zone
+		(net "GND")
+		(layer "In1.Cu")
+		(name "GND plane")
+		(hatch edge 0.5)
+		(connect_pads thru_hole_only
+			(clearance 0.3)
+		)
+		(min_thickness 0.25)
+		(fill yes
+			(thermal_gap 0.5)
+			(thermal_bridge_width 0.5)
+			(island_removal_mode 1)
+		)
+		(polygon
+			(pts
+				(xy 100.3 100.3) (xy 269.7 100.3) (xy 269.7 219.7) (xy 100.3 219.7)
+			)
+		)
+	)
+	(zone
+		(net "+3V3")
+		(layer "In2.Cu")
+		(name "+3V3 plane")
+		(hatch edge 0.5)
+		(connect_pads thru_hole_only
+			(clearance 0.3)
+		)
+		(min_thickness 0.25)
+		(fill yes
+			(thermal_gap 0.5)
+			(thermal_bridge_width 0.5)
+			(island_removal_mode 1)
+		)
+		(polygon
+			(pts
+				(xy 100.3 100.3) (xy 159.75 100.3) (xy 159.75 172.25) (xy 269.7 172.25) (xy 269.7 219.7) (xy 100.3 219.7)
+			)
+		)
+	)
+	(zone
+		(net "+5V")
+		(layer "In2.Cu")
+		(name "+5V plane")
+		(hatch edge 0.5)
+		(connect_pads thru_hole_only
+			(clearance 0.3)
+		)
+		(min_thickness 0.25)
+		(fill yes
+			(thermal_gap 0.5)
+			(thermal_bridge_width 0.5)
+			(island_removal_mode 1)
+		)
+		(polygon
+			(pts
+				(xy 160.25 100.3) (xy 269.7 100.3) (xy 269.7 171.75) (xy 160.25 171.75)
+			)
+		)
 	)
 	(embedded_fonts no)
